File: board/row4.kicad_sch (KiCad schematic)
At the start: 0 parts

Commit message: Connected all rows to MCPs
Other:
- removed sheet HALL_A_1
- removed sheet HALL_B_1
- removed sheet HALL_C_1
- removed sheet HALL_D_1
- removed sheet HALL_E_1
- removed sheet HALL_F_1
- removed sheet HALL_G_1
- removed sheet HALL_H_1
- added sheet HALL_A_4 (hall_sensor.kicad_sch)
- added sheet HALL_B_4 (hall_sensor.kicad_sch)
- added sheet HALL_C_4 (hall_sensor.kicad_sch)
- added sheet HALL_D_4 (hall_sensor.kicad_sch)
- added sheet HALL_E_4 (hall_sensor.kicad_sch)
- added sheet HALL_F_4 (hall_sensor.kicad_sch)
- added sheet HALL_G_4 (hall_sensor.kicad_sch)
- added sheet HALL_H_4 (hall_sensor.kicad_sch)
