File: board/row8.kicad_sch (KiCad schematic)
At the start: 0 parts

Commit message: Connected all rows to MCPs
Other:
- removed sheet HALL_A_1
- removed sheet HALL_B_1
- removed sheet HALL_C_1
- removed sheet HALL_D_1
- removed sheet HALL_E_1
- removed sheet HALL_F_1
- removed sheet HALL_G_1
- removed sheet HALL_H_1
- added sheet HALL_A_8 (hall_sensor.kicad_sch)
- added sheet HALL_B_8 (hall_sensor.kicad_sch)
- added sheet HALL_C_8 (hall_sensor.kicad_sch)
- added sheet HALL_D_8 (hall_sensor.kicad_sch)
- added sheet HALL_E_8 (hall_sensor.kicad_sch)
- added sheet HALL_F_8 (hall_sensor.kicad_sch)
- added sheet HALL_G_8 (hall_sensor.kicad_sch)
- added sheet HALL_H_8 (hall_sensor.kicad_sch)
